Commit message: save

File: catkin_ws/src/kit_agv_description/urdf/kit_agv.urdf.xacro (robot description, xacro)
@@ -39,5 +39,5 @@
     <origin xyz="-0.384099 0.22035 0" rpy="3.14 0 3.14"/>
   </joint>
-  <link name="wheel_right_link">
+  <!-- <link name="wheel_right_link">
     <visual>
       <origin xyz="0 0 0" rpy="1.57 0 0"/>
@@ -68,5 +68,5 @@
     <origin xyz="0.0 0.255 0.171" rpy="0 0 0"/>
     <axis xyz="0 0 1"/>
-  </joint>
+  </joint> -->
   <link name="base_link">
     <visual>
